Commit message: Gazebo Rviz integration complete

File: cry_braccio_description/urdf/braccio_arm.urdf (robot description, URDF)
Before this commit: robot braccio, 11 links, 10 joints
Links:
- link base_link: mass 1 -> 0.1
- link braccio_base_link: mass 1 -> 0.1
- link elbow_link: mass 1 -> 0.1
- link left_gripper_link: mass 1 -> 0.1
- link right_gripper_link: mass 1 -> 0.1
- link shoulder_link: mass 1 -> 0.1
- link wrist_pitch_link: mass 1 -> 0.1
- link wrist_roll_link: mass 1 -> 0.1
Joints:
- joint camera_joint: parent left_gripper_link -> wrist_roll_link
- joint ir_joint: origin xyz=0.0 0 0.01 rpy=0 0 0 -> xyz=0.0 0 0.01 rpy=5 0 3
